File: PCB/TVC_Rocket-PCB/TVC_Rocket-PCB.kicad_sch (KiCad schematic)
At the start: 10 parts, among them J1 MPU_6050-Breakout, J2 UBEC_convertor-connection, U1 Teensy4.1, U3 MS5611-01BA

Commit message: pcb updates
Parts:
- U1: footprint (none) -> teensy4.1:teensy4.1
Changed lines of the file:
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@@
 			)
 		)
-		(property "Footprint" ""
+		(property "Footprint" "teensy4.1:teensy4.1"
 			(at 133.35 106.68 0)
 			(hide yes)
